File: kicad/juubo_left.kicad_pcb (KiCad board)
At the start: 2 copper layers, 145.6 x 125.5 mm, 42 parts

Commit message: Add all ergogen files
Parts:
- moved REF** 2.54 mm to (195.6, 86.4)
- moved REF** 2.54 mm to (198.1, 86.4)
Changed lines of the file:
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@@
   )
   (footprint "Resistor_SMD:R_0201_0603Metric_Pad0.64x0.40mm_HandSolder" (layer "F.Cu")
-    (at 198.12 86.36 90)
+    (at 195.58 86.36 90)
     (descr "Resistor SMD 0201 (0603 Metric), square (rectangular) end terminal, IPC_7351 nominal with elongated pad for handsoldering. (Body size source: https://www.vishay.com/docs/20052/crcw0201e3.pdf), generated with kicad-footprint-generator")
     (tags "resistor handsolder")
@@
   )
   (footprint "Resistor_SMD:R_0201_0603Metric_Pad0.64x0.40mm_HandSolder" (layer "F.Cu")
-    (at 200.66 86.36 90)
+    (at 198.12 86.36 90)
     (descr "Resistor SMD 0201 (0603 Metric), square (rectangular) end terminal, IPC_7351 nominal with elongated pad for handsoldering. (Body size source: https://www.vishay.com/docs/20052/crcw0201e3.pdf), generated with kicad-footprint-generator")
     (tags "resistor handsolder")
