File: kicad_final/juubo_right_final.kicad_pcb (KiCad board)
At the start: 2 copper layers, 145.6 x 125.5 mm, 50 parts

Commit message: Add qmk, gerber, kicad files
Connections:
- MCU1 pad 13: P1 -> GND
Routing:
- net GND: track 109.0 -> 120.2 mm
Other:
- board text added: "juubo_right rev 1.0"
Changed lines of the file:
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@@
       (outputformat 1)
       (mirror false)
-      (drillshape 1)
+      (drillshape 0)
       (scaleselection 1)
-      (outputdirectory "")
+      (outputdirectory "../gerbers/juubo_right_final")
     )
   )
@@
   (net 34 "VCC")
   (net 35 "P18")
-  (net 36 "P1")
-  (net 37 "P0")
-  (net 38 "P2")
-  (net 39 "P3")
-  (net 40 "P9")
-  (net 41 "B+")
+  (net 36 "P0")
+  (net 37 "P2")
+  (net 38 "P3")
+  (net 39 "P9")
+  (net 40 "B+")
   (footprint "E73:SPDT_C128955" (layer "F.Cu")
     (at 291.952306 52.309506)
@@
       (net 32 "RAW"))
     (pad "2" smd rect (at 0.75 2.075) (size 0.9 1.25) (layers "B.Cu" "B.Paste" "B.Mask")
-      (net 41 "B+"))
+      (net 40 "B+"))
     (pad "3" smd rect (at 2.25 2.075) (size 0.9 1.25) (layers "B.Cu" "B.Paste" "B.Mask"))
   )
@@
       (net 34 "VCC"))
     (pad "2" thru_hole oval (at 0 10.2 90) (size 1.6 2.2) (drill oval 0.9 1.5) (layers "*.Cu" "*.Mask")
-      (net 38 "P2"))
+      (net 37 "P2"))
     (pad "3" thru_hole oval (at 0 6.2 90) (size 1.6 2.2) (drill oval 0.9 1.5) (layers "*.Cu" "*.Mask")
-      (net 39 "P3"))
+      (net 38 "P3"))
     (pad "4" thru_hole oval (at 0 3.2 90) (size 1.6 2.2) (drill oval 0.9 1.5) (layers "*.Cu" "*.Mask")
       (net 2 "GND"))
@@
       (stroke (width 0.15) (type solid)) (layer "F.SilkS"))
     (pad "1" thru_hole rect (at -1 0 180) (size 1.2 1.7) (drill 0.75) (layers "*.Cu" "*.Mask")
-      (net 41 "B+"))
+      (net 40 "B+"))
     (pad "2" thru_hole oval (at 1 0 180) (size 1.2 1.7) (drill 0.75) (layers "*.Cu" "*.Mask")
       (net 2 "GND"))
@@
       (net 31 "P10"))
     (pad "13" thru_hole circle (at -13.97 -7.62) (size 1.7526 1.7526) (drill 1.0922) (layers "*.Cu" "*.SilkS" "*.Mask")
-      (net 36 "P1"))
+      (net 2 "GND"))
     (pad "14" thru_hole circle (at -11.43 -7.62) (size 1.7526 1.7526) (drill 1.0922) (layers "*.Cu" "*.SilkS" "*.Mask")
-      (net 37 "P0"))
+      (net 36 "P0"))
     (pad "15" thru_hole circle (at -8.89 -7.62) (size 1.7526 1.7526) (drill 1.0922) (layers "*.Cu" "*.SilkS" "*.Mask")
       (net 2 "GND"))
@@
       (net 2 "GND"))
     (pad "17" thru_hole circle (at -3.81 -7.62) (size 1.7526 1.7526) (drill 1.0922) (layers "*.Cu" "*.SilkS" "*.Mask")
-      (net 38 "P2"))
+      (net 37 "P2"))
     (pad "18" thru_hole circle (at -1.27 -7.62) (size 1.7526 1.7526) (drill 1.0922) (layers "*.Cu" "*.SilkS" "*.Mask")
-      (net 39 "P3"))
+      (net 38 "P3"))
     (pad "19" thru_hole circle (at 1.27 -7.62) (size 1.7526 1.7526) (drill 1.0922) (layers "*.Cu" "*.SilkS" "*.Mask")
       (net 5 "P4"))
@@
       (net 21 "P8"))
     (pad "24" thru_hole circle (at 13.97 -7.62) (size 1.7526 1.7526) (drill 1.0922) (layers "*.Cu" "*.SilkS" "*.Mask")
-      (net 40 "P9"))
+      (net 39 "P9"))
   )
   (footprint "ComboDiode" (layer "F.Cu")
@@
       (net 34 "VCC") (solder_mask_margin 0.102))
     (pad "2" smd rect (at 0.512 0 270) (size 0.475 0.5) (layers "B.Cu" "B.Paste" "B.Mask")
-      (net 39 "P3") (solder_mask_margin 0.102))
+      (net 38 "P3") (solder_mask_margin 0.102))
   )
   (footprint "RES_ERJ2RKF4701X" (layer "B.Cu")
@@
       (net 34 "VCC") (solder_mask_margin 0.102))
     (pad "2" smd rect (at 0.512 0 270) (size 0.475 0.5) (layers "B.Cu" "B.Paste" "B.Mask")
-      (net 38 "P2") (solder_mask_margin 0.102))
+      (net 37 "P2") (solder_mask_margin 0.102))
   )
   (gr_arc (start 274.733342 125.090784) (mid 274.433962 126.550834) (end 273.620867 127.799935)
@@
   (gr_line (start 281.877228 167.351618) (end 333.944592 133.726364)
     (stroke (width 0.15) (type solid)) (layer "Edge.Cuts"))
+  (gr_text "juubo_right rev 1.0" (at 348.7 111.2) (layer "F.SilkS")
+    (effects (font (size 1 1) (thickness 0.1)) (justify left bottom))
+  )
   (segment (start 282.6 84.4) (end 282.6 71.826309) (width 0.25) (layer "F.Cu") (net 1))
   (segment (start 282.6 71.826309) (end 284.332304 70.094005) (width 0.25) (layer "F.Cu") (net 1))
@@
   (segment (start 298.832305 88.377889) (end 294.854416 84.4) (width 0.25) (layer "F.Cu") (net 1))
   (segment (start 281.330799 57.394005) (end 284.332304 57.394005) (width 0.25) (layer "F.Cu") (net 2))
+  (segment (start 296.234005 59.934005) (end 299.572304 59.934005) (width 0.25) (layer "F.Cu") (net 2))
   (segment (start 289.412304 62.474005) (end 284.332304 57.394005) (width 0.25) (layer "F.Cu") (net 2))
+  (segment (start 297.645995 54.854005) (end 296 56.5) (width 0.25) (layer "F.Cu") (net 2))
   (segment (start 299.572304 62.474005) (end 299.572304 59.934005) (width 0.25) (layer "F.Cu") (net 2))
+  (segment (start 296 59.5) (end 295.9 59.6) (width 0.25) (layer "F.Cu") (net 2))
+  (segment (start 296 56.5) (end 296 59.5) (width 0.25) (layer "F.Cu") (net 2))
   (segment (start 281.124804 57.6) (end 281.330799 57.394005) (width 0.25) (layer "F.Cu") (net 2))
   (segment (start 281.124804 54.809003) (end 281.124804 57.6) (width 0.25) (layer "F.Cu") (net 2))
   (segment (start 281.124804 57.6) (end 281.124804 61.009003) (width 0.25) (layer "F.Cu") (net 2))
+  (segment (start 299.572304 54.854005) (end 297.645995 54.854005) (width 0.25) (layer "F.Cu") (net 2))
   (segment (start 299.572304 62.474005) (end 289.412304 62.474005) (width 0.25) (layer "F.Cu") (net 2))
+  (segment (start 295.9 59.6) (end 296.234005 59.934005) (width 0.25) (layer "F.Cu") (net 2))
   (segment (start 290.952304 93.026507) (end 290.952304 64.014005) (width 0.25) (layer "B.Cu") (net 2))
   (segment (start 288.8 103.969002) (end 296.332305 103.969002) (width 0.25) (layer "B.Cu") (net 2))
@@
   (segment (start 287.442306 93.304005) (end 287.442306 87.642306) (width 0.25) (layer "B.Cu") (net 34))
   (segment (start 287.3 87.5) (end 285.637009 85.837009) (width 0.25) (layer "B.Cu") (net 34))
-  (segment (start 294.4 89) (end 294.4 86.8) (width 0.25) (layer "F.Cu") (net 38))
-  (segment (start 286.017306 89.029005) (end 294.370995 89.029005) (width 0.25) (layer "F.Cu") (net 38))
-  (segment (start 294.370995 89.029005) (end 294.4 89) (width 0.25) (layer "F.Cu") (net 38))
-  (via (at 294.4 86.8) (size 0.8) (drill 0.4) (layers "F.Cu" "B.Cu") (net 38))
-  (segment (start 294.4 86.8) (end 294.4 68) (width 0.25) (layer "B.Cu") (net 38))
-  (segment (start 283.84931 86.861009) (end 286.017306 89.029005) (width 0.25) (layer "B.Cu") (net 38))
-  (segment (start 294.4 68) (end 297.385995 65.014005) (width 0.25) (layer "B.Cu") (net 38))
-  (segment (start 283.569806 86.861009) (end 283.84931 86.861009) (width 0.25) (layer "B.Cu") (net 38))
-  (segment (start 297.385995 65.014005) (end 299.572304 65.014005) (width 0.25) (layer "B.Cu") (net 38))
-  (segment (start 282.017306 89.029005) (end 283.708296 89.029005) (width 0.25) (layer "F.Cu") (net 39))
-  (segment (start 295.4 90.4) (end 295.4 86.2) (width 0.25) (layer "F.Cu") (net 39))
-  (segment (start 283.708296 89.029005) (end 285.079291 90.4) (width 0.25) (layer "F.Cu") (net 39))
-  (segment (start 285.079291 90.4) (end 295.4 90.4) (width 0.25) (layer "F.Cu") (net 39))
-  (via (at 295.4 86.2) (size 0.8) (drill 0.4) (layers "F.Cu" "B.Cu") (net 39))
-  (segment (start 281.664801 88.6765) (end 282.017306 89.029005) (width 0.25) (layer "B.Cu") (net 39))
-  (segment (start 295.4 86.2) (end 295.4 71.726309) (width 0.25) (layer "B.Cu") (net 39))
-  (segment (start 295.4 71.726309) (end 299.572304 67.554005) (width 0.25) (layer "B.Cu") (net 39))
-  (segment (start 281.664801 86.861005) (end 281.664801 88.6765) (width 0.25) (layer "B.Cu") (net 39))
-  (segment (start 292.952304 54.634504) (end 292.702306 54.384506) (width 0.25) (layer "B.Cu") (net 41))
-  (segment (start 292.952304 93.026507) (end 292.952304 54.634504) (width 0.25) (layer "B.Cu") (net 41))
+  (segment (start 294.4 89) (end 294.4 86.8) (width 0.25) (layer "F.Cu") (net 37))
+  (segment (start 286.017306 89.029005) (end 294.370995 89.029005) (width 0.25) (layer "F.Cu") (net 37))
+  (segment (start 294.370995 89.029005) (end 294.4 89) (width 0.25) (layer "F.Cu") (net 37))
+  (via (at 294.4 86.8) (size 0.8) (drill 0.4) (layers "F.Cu" "B.Cu") (net 37))
+  (segment (start 294.4 86.8) (end 294.4 68) (width 0.25) (layer "B.Cu") (net 37))
+  (segment (start 283.84931 86.861009) (end 286.017306 89.029005) (width 0.25) (layer "B.Cu") (net 37))
+  (segment (start 294.4 68) (end 297.385995 65.014005) (width 0.25) (layer "B.Cu") (net 37))
+  (segment (start 283.569806 86.861009) (end 283.84931 86.861009) (width 0.25) (layer "B.Cu") (net 37))
+  (segment (start 297.385995 65.014005) (end 299.572304 65.014005) (width 0.25) (layer "B.Cu") (net 37))
+  (segment (start 282.017306 89.029005) (end 283.708296 89.029005) (width 0.25) (layer "F.Cu") (net 38))
+  (segment (start 295.4 90.4) (end 295.4 86.2) (width 0.25) (layer "F.Cu") (net 38))
+  (segment (start 283.708296 89.029005) (end 285.079291 90.4) (width 0.25) (layer "F.Cu") (net 38))
+  (segment (start 285.079291 90.4) (end 295.4 90.4) (width 0.25) (layer "F.Cu") (net 38))
+  (via (at 295.4 86.2) (size 0.8) (drill 0.4) (layers "F.Cu" "B.Cu") (net 38))
+  (segment (start 281.664801 88.6765) (end 282.017306 89.029005) (width 0.25) (layer "B.Cu") (net 38))
+  (segment (start 295.4 86.2) (end 295.4 71.726309) (width 0.25) (layer "B.Cu") (net 38))
+  (segment (start 295.4 71.726309) (end 299.572304 67.554005) (width 0.25) (layer "B.Cu") (net 38))
+  (segment (start 281.664801 86.861005) (end 281.664801 88.6765) (width 0.25) (layer "B.Cu") (net 38))
+  (segment (start 292.952304 54.634504) (end 292.702306 54.384506) (width 0.25) (layer "B.Cu") (net 40))
+  (segment (start 292.952304 93.026507) (end 292.952304 54.634504) (width 0.25) (layer "B.Cu") (net 40))
 )
