File: v2/pcbs/juubo_left _unrouted.kicad_pcb (KiCad board)
At the start: 2 copper layers, 165.7 x 126.6 mm, 53 parts

Commit message: add nice_view, move jst to side, make hole to mcu cover for display
Parts:
- added DISP1: , ceoloide:display_nice_view, F.Cu at (218.3, 71.9)
- moved JST1 13.6 mm to (231.3, 84.8), turned to -180 degrees
Other:
- net class Default removed
