File: v2/pcbs/juubo_right_unfinished.kicad_pcb (KiCad board)
At the start: 2 copper layers, 165.7 x 126.6 mm, 54 parts

Commit message: fix right half row nets
Connections:
- D10 pad 1: P10 -> P14
- D13 pad 1: P10 -> P14
- D16 pad 1: P10 -> P14
- D18 pad 1: P14 -> P10
- D19 pad 1: P14 -> P10
- D2 pad 1: P10 -> P14
- D20 pad 1: P14 -> P10
- D4 pad 1: P10 -> P14
- D7 pad 1: P10 -> P14
